File: STM8_PWM_485.sch (KiCad schematic (older format))
At the start: 30 parts, among them P1 SWIM, P2 PWR, P3 PWM_1, P4 PWM_485, P5 485_EN, U1 nRF24L01_12x18mm, U2 STM8S103K3, U3 MC78M05CDT, U4 AMS1117, U5 MAX487

Commit message: hange to STM32
Parts:
- removed C2: 100n, Capacitors_SMD:C_0805, symbol C_Cer_SMD_0805
- removed C3: 1u, Capacitors_SMD:C_0805, symbol C_Cer_SMD_0805
- removed U2: STM8S103K3, Housings_QFP:LQFP-32_7x7mm_Pitch0.8mm, symbol STM8S103K3
- added C2: 100n, Capacitors_SMD:C_0805, symbol C_Cer_SMD_0603
- added P6: 485, Pin_Headers:Pin_Header_Straight_1x04_Pitch2.54mm, symbol CONN_01X04
- added R11: 10K, Resistors_SMD:R_0805, symbol R_SMD_0805
- added U2: STM32F030K6, Housings_QFP:LQFP-32_7x7mm_Pitch0.8mm, symbol STM32F030K6
- P1: value SWIM -> SWD
- P4: value PWM_485 -> PWM; footprint Pin_Headers:Pin_Header_Straight_1x08_Pitch2.54mm -> Pin_Headers:Pin_Header_Straight_1x09_Pitch2.54mm; symbol CONN_01X08 -> CONN_01X09
Connections:
- net labels added: BOOT0, Button1, LED, PWM_7, PWM_8, SWCLK, SWDIO
- net labels removed: AD2, AD3, SWIM
- wire segments 126 -> 140
- no-connect marks 10 -> 6
Other:
- moved on the sheet: C1, C4, P1, P2, U1

Commit message: PCB UPdate
Parts:
- added D2: ACT, LEDs:LED_0805, symbol Led_Small
- added R12: 1K, Resistors_SMD:R_0805, symbol R_SMD_0805
- added R13: 10K, Resistors_SMD:R_0805, symbol R_SMD_0805
- added SW1: SW, Pin_Headers:Pin_Header_Straight_1x02_Pitch2.00mm, symbol SW_PUSH_SMALL
Connections:
- net labels added: SW1
- net labels removed: Button1
- wire segments 140 -> 148
- no-connect marks 6 -> 4
Other:
- moved on the sheet: C2, R1, R2, R3, R4, R5

Commit message: Update
Parts:
- added C3: 10u, Capacitors_SMD:C_0805, symbol C_Cer_SMD_0805
- C4: footprint Capacitors_SMD:C_0603 -> Capacitors_SMD:C_0805
- R1, R7: value 10k -> 10K
- R11, R13, R4: footprint Resistors_SMD:R_0805 -> Resistors_SMD:R_0603
Connections:
- wire segments 148 -> 150
Changed lines of the file:
@@
 LIBS:contrib
 LIBS:valves
-LIBS:BK_STM8
-LIBS:BK_Common
-LIBS:BK_LED_Drivers
 LIBS:stm32
 LIBS:STM8_PWM_485-cache
@@
 P 3300 6500
 F 0 "R7" H 3330 6520 50  0000 L CNN
-F 1 "10k" H 3330 6460 50  0000 L CNN
+F 1 "10K" H 3330 6460 50  0000 L CNN
 F 2 "Resistors_SMD:R_0603" H 3350 6350 50  0001 C CNN
 F 3 "" H 3300 6500 50  0000 C CNN
@@
 P 1300 1525
 F 0 "R1" H 1330 1545 50  0000 L CNN
-F 1 "10k" H 1330 1485 50  0000 L CNN
+F 1 "10K" H 1330 1485 50  0000 L CNN
 F 2 "Resistors_SMD:R_0603" H 1350 1375 50  0001 C CNN
 F 3 "" H 1300 1525 50  0000 C CNN
@@
 F 0 "C4" H 5285 2620 50  0000 L CNN
 F 1 "100n" H 5285 2470 50  0000 L CNN
-F 2 "Capacitors_SMD:C_0603" H 5275 2400 50  0001 C CNN
+F 2 "Capacitors_SMD:C_0805" H 5275 2400 50  0001 C CNN
 F 3 "" H 5275 2550 50  0000 C CNN
 	1    5275 2550
@@
 	3425 3075 3425 3000
 Wire Wire Line
-	3425 3000 3750 3000
-Wire Wire Line
-	3750 3000 3750 3150
-$Comp
-L GND #PWR019
-U 1 1 5951E3AE
-P 3750 3150
-F 0 "#PWR019" H 3750 2900 50  0001 C CNN
-F 1 "GND" H 3750 3000 50  0000 C CNN
-F 2 "" H 3750 3150 50  0000 C CNN
-F 3 "" H 3750 3150 50  0000 C CNN
-	1    3750 3150
-	1    0    0    -1
-$EndComp
+	3425 3000 3950 3000
 Wire Wire Line
 	3925 3925 4225 3925
@@
 	2925 4225 2500 4225
 Wire Wire Line
-	3425 3300 3150 3300
+	3150 3300 3700 3300
 Wire Wire Line
 	3150 3300 3150 3150
 Connection ~ 3425 3300
 $Comp
-L +3.3V #PWR020
+L +3.3V #PWR019
 U 1 1 5951ED83
 P 3150 3150
-F 0 "#PWR020" H 3150 3000 50  0001 C CNN
+F 0 "#PWR019" H 3150 3000 50  0001 C CNN
 F 1 "+3.3V" H 3150 3290 50  0000 C CNN
 F 2 "" H 3150 3150 50  0000 C CNN
@@
 $EndComp
 $Comp
-L GND #PWR021
+L GND #PWR020
 U 1 1 5951F6B2
 P 3425 4575
-F 0 "#PWR021" H 3425 4325 50  0001 C CNN
+F 0 "#PWR020" H 3425 4325 50  0001 C CNN
 F 1 "GND" H 3425 4425 50  0000 C CNN
 F 2 "" H 3425 4575 50  0000 C CNN
@@
 	5800 1600 5250 1600
 $Comp
-L +12V #PWR022
+L +12V #PWR021
 U 1 1 59526015
 P 1950 1325
-F 0 "#PWR022" H 1950 1175 50  0001 C CNN
+F 0 "#PWR021" H 1950 1175 50  0001 C CNN
 F 1 "+12V" H 1950 1465 50  0000 C CNN
 F 2 "" H 1950 1325 50  0000 C CNN
@@
 F 0 "R4" H 1980 1845 50  0000 L CNN
 F 1 "10K" H 1980 1785 50  0000 L CNN
-F 2 "Resistors_SMD:R_0805" H 2000 1675 50  0001 C CNN
+F 2 "Resistors_SMD:R_0603" H 2000 1675 50  0001 C CNN
 F 3 "" H 1950 1825 50  0000 C CNN
 	1    1950 1825
@@
 $EndComp
 $Comp
-L GND #PWR023
+L GND #PWR022
 U 1 1 595261EC
 P 1950 2025
-F 0 "#PWR023" H 1950 1775 50  0001 C CNN
+F 0 "#PWR022" H 1950 1775 50  0001 C CNN
 F 1 "GND" H 1950 1875 50  0000 C CNN
 F 2 "" H 1950 2025 50  0000 C CNN
@@
 $EndComp
 $Comp
-L +3.3V #PWR024
+L +3.3V #PWR023
 U 1 1 595288FE
 P 2650 1325
-F 0 "#PWR024" H 2650 1175 50  0001 C CNN
+F 0 "#PWR023" H 2650 1175 50  0001 C CNN
 F 1 "+3.3V" H 2650 1465 50  0000 C CNN
 F 2 "" H 2650 1325 50  0000 C CNN
@@
 	2650 1625 2650 1725
 $Comp
-L GND #PWR025
+L GND #PWR024
 U 1 1 59528B3A
 P 2650 2025
-F 0 "#PWR025" H 2650 1775 50  0001 C CNN
+F 0 "#PWR024" H 2650 1775 50  0001 C CNN
 F 1 "GND" H 2650 1875 50  0000 C CNN
 F 2 "" H 2650 2025 50  0000 C CNN
@@
 	7700 4625 7700 4500
 $Comp
-L GND #PWR026
+L GND #PWR025
 U 1 1 5951E1DF
 P 7650 4675
-F 0 "#PWR026" H 7650 4425 50  0001 C CNN
+F 0 "#PWR025" H 7650 4425 50  0001 C CNN
 F 1 "GND" H 7650 4525 50  0000 C CNN
 F 2 "" H 7650 4675 50  0000 C CNN
@@
 Connection ~ 7650 4625
 $Comp
-L +3.3V #PWR027
+L +3.3V #PWR026
 U 1 1 5951E90C
 P 5275 2400
-F 0 "#PWR027" H 5275 2250 50  0001 C CNN
+F 0 "#PWR026" H 5275 2250 50  0001 C CNN
 F 1 "+3.3V" H 5275 2540 50  0000 C CNN
 F 2 "" H 5275 2400 50  0000 C CNN
@@
 $EndComp
 $Comp
-L GND #PWR028
+L GND #PWR027
 U 1 1 5951E96B
 P 5275 2700
-F 0 "#PWR028" H 5275 2450 50  0001 C CNN
+F 0 "#PWR027" H 5275 2450 50  0001 C CNN
 F 1 "GND" H 5275 2550 50  0000 C CNN
 F 2 "" H 5275 2700 50  0000 C CNN
@@
 	7600 975  7600 1100
 $Comp
-L +3.3V #PWR029
+L +3.3V #PWR028
 U 1 1 5951F723
 P 7550 900
-F 0 "#PWR029" H 7550 750 50  0001 C CNN
+F 0 "#PWR028" H 7550 750 50  0001 C CNN
 F 1 "+3.3V" H 7550 1040 50  0000 C CNN
 F 2 "" H 7550 900 50  0000 C CNN
@@
 F 0 "R11" H 5030 1670 50  0000 L CNN
 F 1 "10K" H 5030 1610 50  0000 L CNN
-F 2 "Resistors_SMD:R_0805" H 5050 1500 50  0001 C CNN
+F 2 "Resistors_SMD:R_0603" H 5050 1500 50  0001 C CNN
 F 3 "" H 5000 1650 50  0000 C CNN
 	1    5000 1650
@@
 	5000 1800 5800 1800
 $Comp
-L +3.3V #PWR030
+L +3.3V #PWR029
 U 1 1 5952122C
 P 5000 1350
-F 0 "#PWR030" H 5000 1200 50  0001 C CNN
+F 0 "#PWR029" H 5000 1200 50  0001 C CNN
 F 1 "+3.3V" H 5000 1490 50  0000 C CNN
 F 2 "" H 5000 1350 50  0000 C CNN
@@
 $EndComp
 $Comp
-L +5V #PWR031
+L +5V #PWR030
 U 1 1 59528826
 P 1650 4800
-F 0 "#PWR031" H 1650 4650 50  0001 C CNN
+F 0 "#PWR030" H 1650 4650 50  0001 C CNN
 F 1 "+5V" H 1650 4940 50  0000 C CNN
 F 2 "" H 1650 4800 50  0000 C CNN
@@
 $EndComp
 $Comp
-L GND #PWR032
+L GND #PWR031
 U 1 1 595288F0
 P 1650 5150
-F 0 "#PWR032" H 1650 4900 50  0001 C CNN
+F 0 "#PWR031" H 1650 4900 50  0001 C CNN
 F 1 "GND" H 1650 5000 50  0000 C CNN
 F 2 "" H 1650 5150 50  0000 C CNN
@@
 $EndComp
 $Comp
-L GND #PWR033
+L GND #PWR032
 U 1 1 59521008
 P 3375 2025
-F 0 "#PWR033" H 3375 1775 50  0001 C CNN
+F 0 "#PWR032" H 3375 1775 50  0001 C CNN
 F 1 "GND" H 3375 1875 50  0000 C CNN
 F 2 "" H 3375 2025 50  0000 C CNN
@@
 $EndComp
 $Comp
-L GND #PWR034
+L GND #PWR033
 U 1 1 595279E7
 P 4025 2025
-F 0 "#PWR034" H 4025 1775 50  0001 C CNN
+F 0 "#PWR033" H 4025 1775 50  0001 C CNN
 F 1 "GND" H 4025 1875 50  0000 C CNN
 F 2 "" H 4025 2025 50  0000 C CNN
@@
 F 0 "R13" H 4055 1845 50  0000 L CNN
 F 1 "10K" H 4055 1785 50  0000 L CNN
-F 2 "Resistors_SMD:R_0805" H 4075 1675 50  0001 C CNN
+F 2 "Resistors_SMD:R_0603" H 4075 1675 50  0001 C CNN
 F 3 "" H 4025 1825 50  0000 C CNN
 	1    4025 1825
@@
 	4025 1625 4025 1725
 $Comp
-L +3.3V #PWR035
+L +3.3V #PWR034
 U 1 1 59527E4E
 P 3825 1350
-F 0 "#PWR035" H 3825 1200 50  0001 C CNN
+F 0 "#PWR034" H 3825 1200 50  0001 C CNN
 F 1 "+3.3V" H 3825 1490 50  0000 C CNN
 F 2 "" H 3825 1350 50  0000 C CNN
@@
 Text Label 3675 1675 0    60   ~ 0
 SW1
+$Comp
+L C_Cer_SMD_0805 C3
+U 1 1 59525711
+P 3700 3175
+F 0 "C3" H 3710 3245 50  0000 L CNN
+F 1 "10u" H 3710 3095 50  0000 L CNN
+F 2 "Capacitors_SMD:C_0805" H 3700 3025 50  0001 C CNN
+F 3 "" H 3700 3175 50  0000 C CNN
+	1    3700 3175
+	1    0    0    -1
+$EndComp
+Wire Wire Line
+	3700 3300 3700 3275
+Wire Wire Line
+	3700 3075 3700 3000
+Connection ~ 3700 3000
+$Comp
+L GND #PWR035
+U 1 1 595267B8
+P 3950 3300
+F 0 "#PWR035" H 3950 3050 50  0001 C CNN
+F 1 "GND" H 3950 3150 50  0000 C CNN
+F 2 "" H 3950 3300 50  0000 C CNN
+F 3 "" H 3950 3300 50  0000 C CNN
+	1    3950 3300
+	1    0    0    -1
+$EndComp
+Wire Wire Line
+	3950 3000 3950 3300
 $EndSCHEMATC
